File: PCB/NAL-NIMT-2.kicad_sch (KiCad schematic)
At the start: 27 parts

Commit message: PCB Checkpoint
Parts:
- added D138: WS2812B, PCM_JLCPCB:LED-SMD_4P-L1.6-W1.5_XL-1615RGBC-WS2812B, symbol PCM_JLCPCB-Extended:LED, WS2812B, 1615
- renumbered D138 to D139, D139 to D140, D140 to D141, D141 to D142, D142 to D143, D143 to D144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
Connections:
- net +5V: now also D138.2 (VDD)
- net GND: now also D138.3 (GND)
- net at D139.4 (DIN): now also D138.1 (DOUT); no longer D137.1 (DOUT)
- new net: D137.1 (DOUT), D138.4 (DIN)
Other:
- note removed: "Grafton"
