File: PCB/NAL-NIMT-3.kicad_sch (KiCad schematic)
At the start: 27 parts

Commit message: PCB Checkpoint
Parts:
- renumbered D165 to D166, D166 to D167, D167 to D168, D168 to D169, D169 to D170, D170 to D171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
