File: PCB/NAL-NIMT-4.kicad_sch (KiCad schematic)
At the start: 19 parts

Commit message: PCB Checkpoint
Parts:
- renumbered D192 to D193, D193 to D194, D194 to D195, D195 to D196, D196 to D197, D197 to D198, D198 to D199, D199 to D200, D200 to D201, D201 to D202, D202 to D203, D203 to D204, D204 to D205, D205 to D206, D206 to D207, D207 to D208
Changed lines of the file:
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@@
 		(dnp no)
 		(fields_autoplaced yes)
-		(property "Reference" "D194"
+		(property "Reference" "D195"
 			(at 96.6976 21.6934 0)
 			(effects
@@
 			(project "Auckland-LED-Train-Map"
 				(path "/ab288f7d-a01b-40d1-8b79-fa22fb371f45/081abeee-8e28-48da-a70f-ee01407c3b3b/2bdc9a9d-cd00-4f56-a25d-ca3212db160a/7ea0119b-7e3e-4b22-b10c-5193e6e42080/6bdd3fec-8e69-4213-b97d-b714dd907def"
-					(reference "D194")
+					(reference "D195")
 					(unit 1)
 				)
@@
 		(dnp no)
 		(fields_autoplaced yes)
-		(property "Reference" "D200"
+		(property "Reference" "D201"
 			(at 233.8576 21.6934 0)
 			(effects
@@
 			(project "Auckland-LED-Train-Map"
 				(path "/ab288f7d-a01b-40d1-8b79-fa22fb371f45/081abeee-8e28-48da-a70f-ee01407c3b3b/2bdc9a9d-cd00-4f56-a25d-ca3212db160a/7ea0119b-7e3e-4b22-b10c-5193e6e42080/6bdd3fec-8e69-4213-b97d-b714dd907def"
-					(reference "D200")
+					(reference "D201")
 					(unit 1)
 				)
@@
 		(dnp no)
 		(fields_autoplaced yes)
-		(property "Reference" "D192"
+		(property "Reference" "D193"
 			(at 50.9776 21.6934 0)
 			(effects
@@
 			(project "Auckland-LED-Train-Map"
 				(path "/ab288f7d-a01b-40d1-8b79-fa22fb371f45/081abeee-8e28-48da-a70f-ee01407c3b3b/2bdc9a9d-cd00-4f56-a25d-ca3212db160a/7ea0119b-7e3e-4b22-b10c-5193e6e42080/6bdd3fec-8e69-4213-b97d-b714dd907def"
-					(reference "D192")
+					(reference "D193")
 					(unit 1)
 				)
@@
 		(dnp no)
 		(fields_autoplaced yes)
-		(property "Reference" "D201"
+		(property "Reference" "D202"
 			(at 50.9776 54.7134 0)
 			(effects
@@
 			(project "Auckland-LED-Train-Map"
 				(path "/ab288f7d-a01b-40d1-8b79-fa22fb371f45/081abeee-8e28-48da-a70f-ee01407c3b3b/2bdc9a9d-cd00-4f56-a25d-ca3212db160a/7ea0119b-7e3e-4b22-b10c-5193e6e42080/6bdd3fec-8e69-4213-b97d-b714dd907def"
-					(reference "D201")
+					(reference "D202")
 					(unit 1)
 				)
@@
 		(dnp no)
 		(fields_autoplaced yes)
-		(property "Reference" "D199"
+		(property "Reference" "D200"
 			(at 210.9976 21.6934 0)
 			(effects
@@
 			(project "Auckland-LED-Train-Map"
 				(path "/ab288f7d-a01b-40d1-8b79-fa22fb371f45/081abeee-8e28-48da-a70f-ee01407c3b3b/2bdc9a9d-cd00-4f56-a25d-ca3212db160a/7ea0119b-7e3e-4b22-b10c-5193e6e42080/6bdd3fec-8e69-4213-b97d-b714dd907def"
-					(reference "D199")
+					(reference "D200")
 					(unit 1)
 				)
@@
 		(dnp no)
 		(fields_autoplaced yes)
-		(property "Reference" "D202"
+		(property "Reference" "D203"
 			(at 73.8376 54.7134 0)
 			(effects
@@
 			(project "Auckland-LED-Train-Map"
 				(path "/ab288f7d-a01b-40d1-8b79-fa22fb371f45/081abeee-8e28-48da-a70f-ee01407c3b3b/2bdc9a9d-cd00-4f56-a25d-ca3212db160a/7ea0119b-7e3e-4b22-b10c-5193e6e42080/6bdd3fec-8e69-4213-b97d-b714dd907def"
-					(reference "D202")
+					(reference "D203")
 					(unit 1)
 				)
@@
 		(dnp no)
 		(fields_autoplaced yes)
-		(property "Reference" "D195"
+		(property "Reference" "D196"
 			(at 119.5576 21.6934 0)
 			(effects
@@
 			(project "Auckland-LED-Train-Map"
 				(path "/ab288f7d-a01b-40d1-8b79-fa22fb371f45/081abeee-8e28-48da-a70f-ee01407c3b3b/2bdc9a9d-cd00-4f56-a25d-ca3212db160a/7ea0119b-7e3e-4b22-b10c-5193e6e42080/6bdd3fec-8e69-4213-b97d-b714dd907def"
-					(reference "D195")
+					(reference "D196")
 					(unit 1)
 				)
@@
 		(dnp no)
 		(fields_autoplaced yes)
-		(property "Reference" "D206"
+		(property "Reference" "D207"
 			(at 142.4176 85.1934 0)
 			(effects
@@
 			(project "Auckland-LED-Train-Map"
 				(path "/ab288f7d-a01b-40d1-8b79-fa22fb371f45/081abeee-8e28-48da-a70f-ee01407c3b3b/2bdc9a9d-cd00-4f56-a25d-ca3212db160a/7ea0119b-7e3e-4b22-b10c-5193e6e42080/6bdd3fec-8e69-4213-b97d-b714dd907def"
-					(reference "D206")
+					(reference "D207")
 					(unit 1)
 				)
@@
 		(dnp no)
 		(fields_autoplaced yes)
-		(property "Reference" "D196"
+		(property "Reference" "D197"
 			(at 142.4176 21.6934 0)
 			(effects
@@
 			(project "Auckland-LED-Train-Map"
 				(path "/ab288f7d-a01b-40d1-8b79-fa22fb371f45/081abeee-8e28-48da-a70f-ee01407c3b3b/2bdc9a9d-cd00-4f56-a25d-ca3212db160a/7ea0119b-7e3e-4b22-b10c-5193e6e42080/6bdd3fec-8e69-4213-b97d-b714dd907def"
-					(reference "D196")
+					(reference "D197")
 					(unit 1)
 				)
@@
 		(dnp no)
 		(fields_autoplaced yes)
-		(property "Reference" "D204"
+		(property "Reference" "D205"
 			(at 119.5576 54.7134 0)
 			(effects
@@
 			(project "Auckland-LED-Train-Map"
 				(path "/ab288f7d-a01b-40d1-8b79-fa22fb371f45/081abeee-8e28-48da-a70f-ee01407c3b3b/2bdc9a9d-cd00-4f56-a25d-ca3212db160a/7ea0119b-7e3e-4b22-b10c-5193e6e42080/6bdd3fec-8e69-4213-b97d-b714dd907def"
-					(reference "D204")
+					(reference "D205")
 					(unit 1)
 				)
@@
 		(dnp no)
 		(fields_autoplaced yes)
-		(property "Reference" "D198"
+		(property "Reference" "D199"
 			(at 188.1376 21.6934 0)
 			(effects
@@
 			(project "Auckland-LED-Train-Map"
 				(path "/ab288f7d-a01b-40d1-8b79-fa22fb371f45/081abeee-8e28-48da-a70f-ee01407c3b3b/2bdc9a9d-cd00-4f56-a25d-ca3212db160a/7ea0119b-7e3e-4b22-b10c-5193e6e42080/6bdd3fec-8e69-4213-b97d-b714dd907def"
-					(reference "D198")
+					(reference "D199")
 					(unit 1)
 				)
@@
 		(dnp no)
 		(fields_autoplaced yes)
-		(property "Reference" "D193"
+		(property "Reference" "D194"
 			(at 73.8376 21.6934 0)
 			(effects
@@
 			(project "Auckland-LED-Train-Map"
 				(path "/ab288f7d-a01b-40d1-8b79-fa22fb371f45/081abeee-8e28-48da-a70f-ee01407c3b3b/2bdc9a9d-cd00-4f56-a25d-ca3212db160a/7ea0119b-7e3e-4b22-b10c-5193e6e42080/6bdd3fec-8e69-4213-b97d-b714dd907def"
-					(reference "D193")
+					(reference "D194")
 					(unit 1)
 				)
@@
 		(dnp no)
 		(fields_autoplaced yes)
-		(property "Reference" "D205"
+		(property "Reference" "D206"
 			(at 142.4176 54.7134 0)
 			(effects
@@
 			(project "Auckland-LED-Train-Map"
 				(path "/ab288f7d-a01b-40d1-8b79-fa22fb371f45/081abeee-8e28-48da-a70f-ee01407c3b3b/2bdc9a9d-cd00-4f56-a25d-ca3212db160a/7ea0119b-7e3e-4b22-b10c-5193e6e42080/6bdd3fec-8e69-4213-b97d-b714dd907def"
-					(reference "D205")
+					(reference "D206")
 					(unit 1)
 				)
@@
 		(dnp no)
 		(fields_autoplaced yes)
-		(property "Reference" "D197"
+		(property "Reference" "D198"
 			(at 165.2776 21.6934 0)
 			(effects
@@
 			(project "Auckland-LED-Train-Map"
 				(path "/ab288f7d-a01b-40d1-8b79-fa22fb371f45/081abeee-8e28-48da-a70f-ee01407c3b3b/2bdc9a9d-cd00-4f56-a25d-ca3212db160a/7ea0119b-7e3e-4b22-b10c-5193e6e42080/6bdd3fec-8e69-4213-b97d-b714dd907def"
-					(reference "D197")
+					(reference "D198")
 					(unit 1)
 				)
@@
 		(dnp no)
 		(fields_autoplaced yes)
-		(property "Reference" "D207"
+		(property "Reference" "D208"
 			(at 142.4176 115.6734 0)
 			(effects
@@
 			(project "Auckland-LED-Train-Map"
 				(path "/ab288f7d-a01b-40d1-8b79-fa22fb371f45/081abeee-8e28-48da-a70f-ee01407c3b3b/2bdc9a9d-cd00-4f56-a25d-ca3212db160a/7ea0119b-7e3e-4b22-b10c-5193e6e42080/6bdd3fec-8e69-4213-b97d-b714dd907def"
-					(reference "D207")
+					(reference "D208")
 					(unit 1)
 				)
@@
 		(dnp no)
 		(fields_autoplaced yes)
-		(property "Reference" "D203"
+		(property "Reference" "D204"
 			(at 96.6976 54.7134 0)
 			(effects
@@
 			(project "Auckland-LED-Train-Map"
 				(path "/ab288f7d-a01b-40d1-8b79-fa22fb371f45/081abeee-8e28-48da-a70f-ee01407c3b3b/2bdc9a9d-cd00-4f56-a25d-ca3212db160a/7ea0119b-7e3e-4b22-b10c-5193e6e42080/6bdd3fec-8e69-4213-b97d-b714dd907def"
-					(reference "D203")
+					(reference "D204")
 					(unit 1)
 				)
