File: PCB/Onehunga Branch.kicad_sch (KiCad schematic)
At the start: 5 parts

Commit message: PCB Checkpoint
Parts:
- renumbered D151 to D152, D152 to D153, D153 to D154, D154 to D155, D155 to D156
Changed lines of the file:
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@@
 		(dnp no)
 		(fields_autoplaced yes)
-		(property "Reference" "D153"
+		(property "Reference" "D154"
 			(at 104.3176 19.1534 0)
 			(effects
@@
 			(project "Auckland-LED-Train-Map"
 				(path "/ab288f7d-a01b-40d1-8b79-fa22fb371f45/081abeee-8e28-48da-a70f-ee01407c3b3b/2bdc9a9d-cd00-4f56-a25d-ca3212db160a/a86c74e4-a1b6-4c33-bad3-f8f9d437e222"
-					(reference "D153")
+					(reference "D154")
 					(unit 1)
 				)
@@
 		(dnp no)
 		(fields_autoplaced yes)
-		(property "Reference" "D151"
+		(property "Reference" "D152"
 			(at 58.5976 19.1534 0)
 			(effects
@@
 			(project "Auckland-LED-Train-Map"
 				(path "/ab288f7d-a01b-40d1-8b79-fa22fb371f45/081abeee-8e28-48da-a70f-ee01407c3b3b/2bdc9a9d-cd00-4f56-a25d-ca3212db160a/a86c74e4-a1b6-4c33-bad3-f8f9d437e222"
-					(reference "D151")
+					(reference "D152")
 					(unit 1)
 				)
@@
 		(dnp no)
 		(fields_autoplaced yes)
-		(property "Reference" "D155"
+		(property "Reference" "D156"
 			(at 150.0376 19.1534 0)
 			(effects
@@
 			(project "Auckland-LED-Train-Map"
 				(path "/ab288f7d-a01b-40d1-8b79-fa22fb371f45/081abeee-8e28-48da-a70f-ee01407c3b3b/2bdc9a9d-cd00-4f56-a25d-ca3212db160a/a86c74e4-a1b6-4c33-bad3-f8f9d437e222"
-					(reference "D155")
+					(reference "D156")
 					(unit 1)
 				)
@@
 		(dnp no)
 		(fields_autoplaced yes)
-		(property "Reference" "D152"
+		(property "Reference" "D153"
 			(at 81.4576 19.1534 0)
 			(effects
@@
 			(project "Auckland-LED-Train-Map"
 				(path "/ab288f7d-a01b-40d1-8b79-fa22fb371f45/081abeee-8e28-48da-a70f-ee01407c3b3b/2bdc9a9d-cd00-4f56-a25d-ca3212db160a/a86c74e4-a1b6-4c33-bad3-f8f9d437e222"
-					(reference "D152")
+					(reference "D153")
 					(unit 1)
 				)
@@
 		(dnp no)
 		(fields_autoplaced yes)
-		(property "Reference" "D154"
+		(property "Reference" "D155"
 			(at 127.1776 19.1534 0)
 			(effects
@@
 			(project "Auckland-LED-Train-Map"
 				(path "/ab288f7d-a01b-40d1-8b79-fa22fb371f45/081abeee-8e28-48da-a70f-ee01407c3b3b/2bdc9a9d-cd00-4f56-a25d-ca3212db160a/a86c74e4-a1b6-4c33-bad3-f8f9d437e222"
-					(reference "D154")
-					(unit 1)
-				)
+					(reference "D155")
+					(unit 1)
+				)
