File: PCB/STRAND-MNK-1.kicad_sch (KiCad schematic)
At the start: 43 parts

Commit message: PCB Checkpoint
Parts:
- added D304: WS2812B, PCM_JLCPCB:LED-SMD_4P-L1.6-W1.5_XL-1615RGBC-WS2812B, symbol PCM_JLCPCB-Extended:LED, WS2812B, 1615
- renumbered D304 to D305, D305 to D306, D306 to D307, D307 to D308, D308 to D309, D309 to D310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
Connections:
- net +5V: now also D304.2 (VDD)
- net GND: now also D304.3 (GND)
- net at D303.1 (DOUT): now also D304.4 (DIN); no longer D305.4 (DIN)
- new net: D304.1 (DOUT), D305.4 (DIN)
Other:
- moved on the sheet: D300, D301, D302, D303
