File: PCB/STRAND-MNK-2.kicad_sch (KiCad schematic)
At the start: 4 parts

Commit message: PCB Checkpoint
Parts:
- renumbered D340 to D341, D341 to D342, D342 to D343, D343 to D344
Changed lines of the file:
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@@
 		(dnp no)
 		(fields_autoplaced yes)
-		(property "Reference" "D342"
+		(property "Reference" "D343"
 			(at 134.7976 21.6934 0)
 			(effects
@@
 			(project "Auckland-LED-Train-Map"
 				(path "/ab288f7d-a01b-40d1-8b79-fa22fb371f45/dbd0708e-69d8-4d43-bcc7-3988563b469e/e16470c1-e6de-4b7a-8c2a-2890c425ddf6"
-					(reference "D342")
+					(reference "D343")
 					(unit 1)
 				)
@@
 		(dnp no)
 		(fields_autoplaced yes)
-		(property "Reference" "D343"
+		(property "Reference" "D344"
 			(at 157.6576 21.6934 0)
 			(effects
@@
 			(project "Auckland-LED-Train-Map"
 				(path "/ab288f7d-a01b-40d1-8b79-fa22fb371f45/dbd0708e-69d8-4d43-bcc7-3988563b469e/e16470c1-e6de-4b7a-8c2a-2890c425ddf6"
-					(reference "D343")
+					(reference "D344")
 					(unit 1)
 				)
@@
 		(dnp no)
 		(fields_autoplaced yes)
-		(property "Reference" "D341"
+		(property "Reference" "D342"
 			(at 111.9376 21.6934 0)
 			(effects
@@
 			(project "Auckland-LED-Train-Map"
 				(path "/ab288f7d-a01b-40d1-8b79-fa22fb371f45/dbd0708e-69d8-4d43-bcc7-3988563b469e/e16470c1-e6de-4b7a-8c2a-2890c425ddf6"
-					(reference "D341")
+					(reference "D342")
 					(unit 1)
 				)
@@
 		(dnp no)
 		(fields_autoplaced yes)
-		(property "Reference" "D340"
+		(property "Reference" "D341"
 			(at 50.9776 21.6934 0)
 			(effects
@@
 			(project "Auckland-LED-Train-Map"
 				(path "/ab288f7d-a01b-40d1-8b79-fa22fb371f45/dbd0708e-69d8-4d43-bcc7-3988563b469e/e16470c1-e6de-4b7a-8c2a-2890c425ddf6"
-					(reference "D340")
-					(unit 1)
-				)
+					(reference "D341")
+					(unit 1)
+				)
