File: PCB/Auckland-LED-Train-Map.kicad_sch (KiCad schematic)
At the start: 102 parts, among them J1 Prog Connector, Q1 HL3415A, Q2 MMBT3904, U1 XC6206P332MR, U2 ESP32-C3FH4, U3 SN74LVC4245APWR, U4 Connector, USB-TYPE-C-16P, U5 Connector, USB-TYPE-C-16P, X1 40MHz, 15pF

Commit message: PCB Checkpoint
Parts:
- removed C15, C5: 100uF, PCM_JLCPCB:C_1206, symbol PCM_JLCPCB-Capacitors:1206,100uF
- removed H4: ~, PCM_JLCPCB:Hole_Tooling_JLCPCB, symbol PCM_JLCPCB-Manufacturing:Tooling Hole, PCM_JLCPCB, 1.152mm
- added C5: 100uF, PCM_JLCPCB:C_CASE-B-3528-21(mm), symbol PCM_JLCPCB-Capacitors:CASE-B-3528-21(mm),100uF
- added FB1: ~, PCM_JLCPCB:FB_0603, symbol PCM_JLCPCB-Inductors:Ferrite,0603,(2)
- F1: value Polyfuse, 2.5A -> Polyfuse, 2A; footprint Fuse:Fuse_0805_2012Metric_Pad1.15x1.40mm_HandSolder -> Fuse:Fuse_1206_3216Metric; LCSC C2757931 -> C6165195; Manufacturer BHFUSE -> (none); Part BSMD0805L-200 -> (none)
Connections:
- net +3V3: now also C5.1
- net GND: now also C5.2
- net at D2.2, D6.1, D7.1: now also FB1.1; no longer F1.1
- new net: F1.1, FB1.2
Other:
- moved on the sheet: D1, F1

Commit message: PCB Checkpoint
Parts:
- removed C1, C25: 10uF, PCM_JLCPCB:C_0603, symbol PCM_JLCPCB-Capacitors:0603,10uF
- added C1: 10uF, PCM_JLCPCB:C_CASE-A-3216-18(mm), symbol PCM_JLCPCB-Capacitors:CASE-A-3216-18(mm),10uF
Connections:
- net GND: now also C1.2
- net VBUS: now also C1.1

Commit message: Finish V1.1 PCB
Parts:
- removed D3: SRV05-4A, PCM_JLCPCB:SOT-23-6_L2.9-W1.6-P0.95-LS2.9-BL, symbol PCM_JLCPCB-Diode-Packages:Package, SRV05-4A_C20615829
- removed TP10: VBUS, Custom_Footprints:TestPoint_Pad_D1.0mm, symbol Connector:TestPoint
- removed TP11: GND, Custom_Footprints:TestPoint_Pad_D1.0mm, symbol Connector:TestPoint
- removed TP12: WiFi_LED, Custom_Footprints:TestPoint_Pad_D1.0mm, symbol Connector:TestPoint
- removed TP14: Config_LED, Custom_Footprints:TestPoint_Pad_D1.0mm, symbol Connector:TestPoint
- removed TP5: PMOS_Gate, Custom_Footprints:TestPoint_Pad_D1.0mm, symbol Connector:TestPoint
- removed TP6: ALED_5V, Custom_Footprints:TestPoint_Pad_D1.0mm, symbol Connector:TestPoint
- removed TP7: NPN_Gate, Custom_Footprints:TestPoint_Pad_D1.0mm, symbol Connector:TestPoint
- added C15: 100uF, PCM_JLCPCB:C_CASE-B-3528-21(mm), symbol PCM_JLCPCB-Capacitors:CASE-B-3528-21(mm),100uF
- added C25: 10uF, PCM_JLCPCB:C_0402, symbol PCM_JLCPCB-Capacitors:0402,10uF
- R22, R23, R9: value 47kΩ -> 100kΩ; symbol PCM_JLCPCB-Resistors:0402,47kΩ -> PCM_JLCPCB-Resistors:0402,100kΩ; LCSC C25792 -> C25741; Part 0402WGF4702TCE -> 0402WGF1003TCE; Resistance 47kΩ -> 100kΩ; Stock 1134503 -> 4111720
Connections:
- net +3V3: now also C25.1
- net +5V: now also C15.1
- net GND: now also C15.2, C25.2
