File: PCB/Auckland-LED-Train-Map.kicad_pcb (KiCad board)
At the start: 2 copper layers, 249 x 70 mm, 263 parts, among them J1 Prog Connector, Q1 HL3415A, Q2 MMBT3904, U1 XC6206P332MR, U2 ESP32-C3FH4, U3 SN74LVC4245APWR, U4 Connector, USB-TYPE-C-16P, U5 Connector, USB-TYPE-C-16P, X1 40MHz, 15pF

Commit message: Remove firmware folder and update readme
Routing:
- net Net-(D150-DOUT): track 6.51 -> 5.58 mm, vias 3 -> 2
Other:
- board text added: "Solder coming through back on one sample..."
